Commit message: adding gz-brdige

File: crazyflie_ws/src/crazyflie_description/urdf/crazyflie_body.xacro (robot description, xacro)
@@ -90,5 +90,5 @@
     <origin xyz="0.031 -0.031 0.021" rpy="0 0 0"/>
     <axis xyz="0 0 1"/>
-    <limit effort="1.0" velocity="100.0"/>
+    <limit effort="1.0" velocity="120.0"/>
   </joint>
   <joint name="body_to_m2_prop" type="continuous">
@@ -97,5 +97,5 @@
     <origin xyz="-0.031 -0.031 0.021" rpy="0 0 0"/>
     <axis xyz="0 0 1"/>
-    <limit effort="1.0" velocity="100.0"/>
+    <limit effort="1.0" velocity="120.0"/>
   </joint>
   <joint name="body_to_m3_prop" type="continuous">
@@ -104,5 +104,5 @@
     <origin xyz="-0.031 0.031 0.021" rpy="0 0 0"/>
     <axis xyz="0 0 1"/>
-    <limit effort="1.0" velocity="100.0"/>
+    <limit effort="1.0" velocity="120.0"/>
   </joint>
   <joint name="body_to_m4_prop" type="continuous">
@@ -111,5 +111,5 @@
     <origin xyz="0.031 0.031 0.021" rpy="0 0 0"/>
     <axis xyz="0 0 1"/>
-    <limit effort="1.0" velocity="100.0"/>
+    <limit effort="1.0" velocity="120.0"/>
   </joint>
   <gazebo>
